Commit message: ros2_control implemented but tyson is not moving straight

File: Tyson_MK1/ros2_ws/src/tyson_description/urdf/tyson.xacro (robot description, xacro)
@@ -1,4 +1,6 @@
 <?xml version="1.0" ?>
 <robot name="tyson" xmlns:xacro="http://www.ros.org/wiki/xacro">
+<xacro:arg name="use_sim" default="true"/>
+<xacro:property name="use_sim" value="$(arg use_sim)"/>
 <xacro:include filename="$(find tyson_description)/urdf/materials.xacro" />
 <xacro:include filename="$(find tyson_description)/urdf/tyson.ros2control" />

Commit message: working gazebo simgit status issue: collision = mesh file

File: Tyson_MK1/ros2_ws/src/tyson_description/urdf/tyson.xacro (robot description, xacro)
@@ -73,5 +73,5 @@
   </inertial>
   <visual>
-    <origin xyz="-0.208 -0.166 -0.052606" rpy="0 0 0"/>
+    <origin xyz="-0.208 -0.166 -0.053" rpy="0 0 0"/>
     <geometry>
       <mesh filename="file://$(find tyson_description)/meshes/wheel_fl_1.stl" scale="0.001 0.001 0.001"/>
@@ -80,5 +80,5 @@
   </visual>
   <collision>
-    <origin xyz="-0.208 -0.166 -0.052606" rpy="0 0 0"/>
+    <origin xyz="-0.208 -0.166 -0.053" rpy="0 0 0"/>
     <geometry>
       <mesh filename="file://$(find tyson_description)/meshes/wheel_fl_1.stl" scale="0.001 0.001 0.001"/>
@@ -150,5 +150,5 @@
   <parent link="base_link"/>
   <child link="wheel_fr_1"/>
-  <axis xyz="0.0 -1.0 0.0"/>
+  <axis xyz="0.0 1.0 0.0"/>
 </joint>
 <joint name="wheel_rr_joint" type="continuous">
@@ -156,8 +156,8 @@
   <parent link="base_link"/>
   <child link="wheel_rr_1"/>
-  <axis xyz="0.0 -1.0 0.0"/>
+  <axis xyz="0.0 1.0 0.0"/>
 </joint>
 <joint name="wheel_fl_joint" type="continuous">
-  <origin xyz="0.208 0.166 0.052606" rpy="0 0 0"/>
+  <origin xyz="0.208 0.166 0.053" rpy="0 0 0"/>
   <parent link="base_link"/>
   <child link="wheel_fl_1"/>
